File: BalthazarPSU3.kicad_pcb (KiCad board)
At the start: 2 copper layers, 84.8 x 25.4 mm, 87 parts, among them IC1 BQ24193, J1 AudioIN, J2 USB_C_Receptacle_USB2.0, J3 5-15V/3A, J4 AudioOUT, J7 uC host, J8 5V 2A, J9 12V 2A, Q1 IRF7404, Q2 BSS138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

Commit message: Add files via upload
Parts:
- removed H1: MountingHole_Pad, MountingHole:MountingHole_2.2mm_M2_Pad
- H3: value MountingHole_Pad -> hole
- J3: value 5-15V/3A -> 5-15V / 3-5A; footprint TerminalBlock:TerminalBlock_bornier-2_P5.08mm -> Connector_BarrelJack:BarrelJack_Horizontal
- J8: value 5V 2A -> 5V 3A
- moved J3 6.86 mm to (111.0, 62.3)
- moved J2 2.58 mm to (106.9, 70.6)
- moved R16 2.41 mm to (121.3, 70.4)
- moved R19 2.29 mm to (103.1, 74.3)
- moved R28 2.29 mm to (103.1, 76.2)
- moved H3 1.02 mm to (104.0, 80.8)
Connections:
- J3 pad 1: PGND -> VPSU
- J3 pad 2: VPSU -> PGND
Routing:
- net VPSU: track 37.7 -> 30.0 mm
- net VBUS: track 140.2 -> 133.5 mm, vias 8 -> 9
- net PGND: track 127.6 -> 124.3 mm
- net Net-(J2-CC1): track 4.78 -> 7.48 mm
- net Net-(IC1-/PG): track 28.6 -> 31.2 mm
- net Net-(IC1-PSEL): track 27.5 -> 30.1 mm
- net Net-(J2-CC2): track 5.44 -> 4.40 mm
Other:
- board size 84.8 x 25.4 mm -> 85.9 x 25.4 mm
