File: BalthazarPSU3.kicad_sch (KiCad schematic)
At the start: 87 parts

Commit message: Add files via upload
Parts:
- removed U: (no value), symbol Mechanical:MountingHole_Pad
Connections:
- net Earth: now also U.2 (Pin_2); no longer U.1 (Pin_1)
- net VPSU: now also U.1 (Pin_1); no longer U.2 (Pin_2)
Other:
- moved on the sheet: U
Changed lines of the file:
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@@
   (junction (at 110.49 19.05) (diameter 0) (color 0 0 0 0)
   )
-  (junction (at 31.75 116.84) (diameter 0) (color 0 0 0 0)
-  )
   (junction (at 92.71 64.77) (diameter 0) (color 0 0 0 0)
   )
@@
     (stroke (width 0) (type default))
   )
-  (wire (pts (xy 31.75 105.41) (xy 31.75 116.84))
+  (wire (pts (xy 31.75 105.41) (xy 31.75 121.92))
     (stroke (width 0) (type default))
   )
@@
     (stroke (width 0) (type default))
   )
-  (wire (pts (xy 31.75 116.84) (xy 31.75 121.92))
-    (stroke (width 0) (type default))
-  )
   (wire (pts (xy 90.17 105.41) (xy 53.34 105.41))
     (stroke (width 0) (type default))
@@
     (pin "S1")
   )
-  (symbol (lib_id "Connector:Conn_01x02_Female") (at 16.51 76.2 180) (unit 1)
+  (symbol (lib_id "Connector:Conn_01x02_Female") (at 16.51 73.66 0) (mirror y) (unit 1)
     (in_bom yes) (on_board yes)
     (default_instance (reference "U") (unit 1) (value "") (footprint ""))
@@
       (effects (font (size 1.27 1.27)) (justify left))
     )
-    (property "Value" "" (id 1) (at 24.13 71.12 0)
+    (property "Value" "" (id 1) (at 24.13 78.74 0)
       (effects (font (size 1.27 1.27)) (justify left))
     )
-    (property "Footprint" "" (id 2) (at 16.51 76.2 0)
+    (property "Footprint" "" (id 2) (at 16.51 73.66 0)
       (effects (font (size 1.27 1.27)) hide)
     )
-    (property "Datasheet" "~" (id 3) (at 16.51 76.2 0)
+    (property "Datasheet" "~" (id 3) (at 16.51 73.66 0)
       (effects (font (size 1.27 1.27)) hide)
     )
@@
     (pin "2")
   )
-  (symbol (lib_id "Mechanical:MountingHole_Pad") (at 29.21 116.84 90) (unit 1)
-    (in_bom yes) (on_board yes)
-    (default_instance (reference "U") (unit 1) (value "") (footprint ""))
-    (property "Reference" "U" (id 0) (at 24.13 116.84 90)
-      (effects (font (size 1.27 1.27)))
-    )
-    (property "Value" "" (id 1) (at 29.1338 113.1316 90)
-      (effects (font (size 1.27 1.27)) hide)
-    )
-    (property "Footprint" "" (id 2) (at 29.21 116.84 0)
-      (effects (font (size 1.27 1.27)) hide)
-    )
-    (property "Datasheet" "~" (id 3) (at 29.21 116.84 0)
-      (effects (font (size 1.27 1.27)) hide)
-    )
-    (pin "1")
-  )
   (symbol (lib_id "Mechanical:MountingHole_Pad") (at 29.21 121.92 90) (unit 1)
     (in_bom yes) (on_board yes)
@@
       (reference "D7") (unit 1) (value "B320") (footprint "Diode_SMD:D_SMB")
     )
-    (path "/00000000-0000-0000-0000-00005fdfba45"
-      (reference "H1") (unit 1) (value "MountingHole_Pad") (footprint "MountingHole:MountingHole_2.2mm_M2_Pad")
-    )
     (path "/00000000-0000-0000-0000-00005fdff4b2"
       (reference "H3") (unit 1) (value "hole") (footprint "MountingHole:MountingHole_2.2mm_M2_Pad")
@@
     )
     (path "/00000000-0000-0000-0000-00005fb9e4d9"
-      (reference "J3") (unit 1) (value "5-15V / 3-5A") (footprint "TerminalBlock:TerminalBlock_bornier-2_P5.08mm")
+      (reference "J3") (unit 1) (value "5-15V / 3-5A") (footprint "Connector_BarrelJack:BarrelJack_Horizontal")
     )
     (path "/00000000-0000-0000-0000-00005ea6f019"
