File: kicad/BalthazarPSU3.kicad_pcb (KiCad board)
At the start: 4 copper layers, 85.9 x 25.4 mm, 84 parts, among them IC1 BQ24193, J1 AudioIN, J2 USB_C_Receptacle_USB2.0, J3 5-15V / 3-5A, J4 AudioOUT, J7 uC host, J8 5V 3A, J9 12V 2A, Q1 IRF7404, Q2 BSS138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

Commit message: fixing/checking design errors fix #12
Routing:
- net Net-(U3-EN): track 13.2 -> 10.9 mm
- net Net-(U3-L2): track 12.5 -> 10.5 mm, vias 1 -> 0
- net VBUS: track 36.9 -> 35.9 mm, vias 7 -> 5
- net Net-(IC1-REGN): track 24.5 -> 23.7 mm
- net Net-(J4-Pin_1): track 7.92 -> 7.12 mm
- net Net-(U3-PG): track 13.1 -> 13.9 mm
- net 5V: track 12.5 -> 13.2 mm, vias 2 -> 1
- net PGND: track 64.2 -> 63.6 mm
- net 12V: track 7.86 -> 7.49 mm, vias 2 -> 0
- net VSYS: vias 6 -> 5
- net Net-(U3-L1): vias 1 -> 0
- net Net-(IC1-SW): vias 2 -> 1
- removed copper zone on F.Cu, net (none)

Commit message: Improving schematics #5
Connections:
- CBUS1 pad 1: VSYS -> PGND
- CBUS1 pad 2: PGND -> VSYS
Routing:
- net VSYS: track 103.0 -> 106.4 mm, vias 5 -> 6

Commit message: Adding production files fix #8
Connections:
- net Net-(IC1-INT) renamed /INT
- net Net-(IC1-OTG) renamed /OTG
- net Net-(IC1-PSEL) renamed /D+
- net Net-(IC1-SCL) renamed /SCL
- net Net-(IC1-SDA) renamed /SDA
- net Net-(IC1-/CE) renamed /CE
- net Net-(IC1-/PG) renamed /D-
Routing:
- net PGND: track 63.5 -> 64.0 mm
Other:
- board text added: "BALTHAZAR v02"
- board text removed: "BALTHAZAR"
