File: kicad/BalthazarPSU3.kicad_sch (KiCad schematic)
At the start: 84 parts, among them IC1 BQ24193, J1 AudioIN, J2 USB_C_Receptacle_USB2.0, J3 5-15V / 3-5A, J4 AudioOUT, J7 uC host, J8 5V 3A, J9 12V 2A, Q1 IRF7404, Q2 BSS138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

Commit message: Moving more lines
Connections:
- net VSYS: no longer R1.2
- net SCL: now reaches IC1.5 (SCL), J7.2 (Pin_2), R3.1
- net SDA: now reaches IC1.6 (SDA), J7.3 (Pin_3), R2.1
- net INT: now reaches IC1.7 (INT), J7.4 (Pin_4), R1.1
- net CE: now reaches IC1.9 (/CE), J7.5 (Pin_5), R6.1
- net at Q2.3 (D), R17.1: no longer IC1.8 (OTG)
- new net OTG: IC1.8 (OTG)
Other:
- moved on the sheet: R1, R17, R2, R3, R6, R7

Commit message: Moving more lines
Connections:
- net VSYS: now also R1.2
Other:
- moved on the sheet: C25, H3, H4, J3, J7, Q1, Q2, Q3, R17, R38, R39, R40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
